Commit message: Add ROS2 control configuration and joint state publisher updates
- Introduced spm_controllers.yaml for controller management.
- Updated CMakeLists.txt to include std_msgs dependency.
- Enhanced spm_joint_state_publisher to publish commands for forward_position_controller.
- Added launch file for control stack initialization with RViz support.
- Extended robot_core.xacro to define actuated joints for ros2_control.

File: description/robot.urdf.xacro (robot description, xacro)
@@ -2,3 +2,30 @@
 <robot xmlns:xacro="http://www.ros.org/wiki/xacro"  name="robot">
     <xacro:include filename="$(find spm_robot)/description/robot_core.xacro" />
+	<!-- ROS2_CONTROL -->
+	<!-- Only the three base joints are actuated. The *_upper joints are
+	     passive, kinematically coupled through the parallel mechanism (and
+	     through the still-commented-out platform), so they are intentionally
+	     left out of ros2_control: nothing drives them directly, and a
+	     mock/simulated HardwareInterface would just report whatever value
+	     you set, with no coupling to the actuated joints. -->
+	<ros2_control name="SPMSystem" type="system">
+		<hardware>
+			<plugin>mock_components/GenericSystem</plugin>
+		</hardware>
+		<joint name="first_arm_joint">
+			<command_interface name="position"/>
+			<state_interface name="position"/>
+			<state_interface name="velocity"/>
+		</joint>
+		<joint name="second_arm_joint">
+			<command_interface name="position"/>
+			<state_interface name="position"/>
+			<state_interface name="velocity"/>
+		</joint>
+		<joint name="third_arm_joint">
+			<command_interface name="position"/>
+			<state_interface name="position"/>
+			<state_interface name="velocity"/>
+		</joint>
+	</ros2_control>
 </robot>
